Commit message: copy over ms3 code

File: mani_skill2/assets/robots/panda/panda_v2.urdf (robot description, URDF)
Before this commit: robot panda, 13 links, 12 joints
Links:
- added link panda_leftfinger_pad
- added link panda_rightfinger_pad
Joints:
- added joint panda_leftfinger_pad_joint: type fixed, parent panda_leftfinger, child panda_leftfinger_pad, origin xyz=0 0 0.0455 rpy=0 0 0
- added joint panda_rightfinger_pad_joint: type fixed, parent panda_rightfinger, child panda_rightfinger_pad, origin xyz=0 0 0.0455 rpy=0 0 0
