Commit message: Progress: Fetch mobile base

File: mani_skill2/assets/robots/fetch/fetch.urdf (robot description, URDF)
Before this commit: robot fetch, 26 links, 25 joints
Links:
- added link root, mass 0
- added link root_arm_1_link_1, mass 0
- added link root_arm_1_link_2, mass 0
Joints:
- added joint root_x_axis_joint: type prismatic, parent root, child root_arm_1_link_1, axis 1 0 0, limit lower=-10 upper=10 velocity=0.50
- added joint root_y_axis_joint: type prismatic, parent root_arm_1_link_1, child root_arm_1_link_2, axis 0 1 0, limit lower=-10 upper=10 velocity=0.50
- added joint root_z_rotation_joint: type continuous, parent root_arm_1_link_2, child base_link, axis 0 0 1

Commit message: Squashed commit of the following:
commit 27101d4bdc4bd98451ed38d209045b36794288a9
Author: Stone Tao <stonezt2019@gmail.com>
Date:   Tue Jan 23 18:12:03 2024 -0800

    fix some bugs with fetch

File: mani_skill2/assets/robots/fetch/fetch.urdf (robot description, URDF)
Before this commit: robot fetch, 29 links, 28 joints
Joints:
- joint root_x_axis_joint: limit lower=-10 upper=10 velocity=0.50 -> lower=-10 upper=10 effort=100 velocity=0.50
- joint root_y_axis_joint: limit lower=-10 upper=10 velocity=0.50 -> lower=-10 upper=10 effort=100 velocity=0.50

Commit message: GPU Simulated Scenes, New more organized asset locations (#217)
* Fix: some scene manip env issues

* Better fetch cameras

* Fix: disable collisions only on fetch wheels

* Fix: fetch grapsing retval

* Progress: updates to scene-related classes/envs

* Fix: ai2thor scene builder set poses in initialize()

* Fix: ai2thor fetch scene builder ground collisions

* Fix: ai2 sb don't reconfigure by default

* Fix: sb load_actors instead of load_agents

* Trivial: add fetch resting qpos as attr

* Fix: pick_object scene pose setting

* Fix: renderer follows camera

* Fix: options is None

* Fix: fetch body delta pos controller

* Fix: record wrapper options=None by default

* Progress: support for loading navigable positions

* Progress: update base scene builder w/ DexM3 version

* Trivial: add arm camera, more "working" coacd objects

* minor ai2 sb changes

* Trivial: port over everything needed for scene manip testing

* bigger place reward

* Fix: keep x/y/zrot qvel in obs

* Try tune reward

* scale place reward more

* Try lessen place rew

* work

* work

* add bug fix

* Create scene_gpu.py

* Update sequential_task.py

* temp code

* make more objects static

* base empty scene manipulation env

* work

* work

* tests

* work

* more work

* modify benchmark code to support cpu and gpu sim tests

* add lighting?

* work

* articulations

* work

* Update scene_builder.py

* new dataset location

* fix for new dataset paths for some tasks, remove old tasks

* remove scene tasks as they are not done

* work

* work

* fixes

* change some defaults

---------

Co-authored-by: arth-shukla <44527268+arth-shukla@users.noreply.github.com>

File: mani_skill2/assets/robots/fetch/fetch.urdf (robot description, URDF)
Before this commit: robot fetch, 29 links, 28 joints
Joints:
- joint root_x_axis_joint: limit lower=-10 upper=10 effort=100 velocity=0.50 -> lower=-20 upper=20 effort=100 velocity=0.50
- joint root_y_axis_joint: limit lower=-10 upper=10 effort=100 velocity=0.50 -> lower=-20 upper=20 effort=100 velocity=0.50
