Commit message: bug fix, upgrade realsense panda arm with actual real sense camera mesh

File: mani_skill/assets/robots/panda/panda_v3.urdf (robot description, URDF)
Before this commit: robot panda, 15 links, 14 joints
Links:
- link camera_link: geometry collision box size=0.02005 0.099 0.023; visual mesh filename=realsense2_description/meshes/d415.stl
