Commit message: fix a few files

File: mani_skill/assets/robots/unitree_h1/urdf/h1.urdf (robot description, URDF)
Before this commit: robot h1_description, 25 links, 24 joints
Links:
- link torso_link: geometry collision mesh filename=../meshes/torso_link.glb; visual mesh filename=../meshes/torso_link.dae

Commit message: work

File: mani_skill/assets/robots/unitree_h1/urdf/h1.urdf (robot description, URDF)
Before this commit: robot h1_description, 25 links, 24 joints
Links:
- removed link d435_left_imager_link
- removed link d435_rgb_module_link
- removed link mid360_link
- link left_ankle_link: geometry collision mesh filename=../meshes/left_ankle_link.glb; visual mesh filename=../meshes/left_ankle_link.dae
- link left_elbow_link: geometry collision mesh filename=../meshes/left_elbow_link.glb; visual mesh filename=../meshes/left_elbow_link.dae
- link left_hip_pitch_link: geometry collision mesh filename=../meshes/left_hip_pitch_link.glb; visual mesh filename=../meshes/left_hip_pitch_link.dae
- link left_hip_roll_link: geometry collision mesh filename=../meshes/left_hip_roll_link.glb; visual mesh filename=../meshes/left_hip_roll_link.dae
- link left_hip_yaw_link: geometry collision mesh filename=../meshes/left_hip_yaw_link.glb; visual mesh filename=../meshes/left_hip_yaw_link.dae
- link left_knee_link: geometry collision mesh filename=../meshes/left_knee_link.glb; visual mesh filename=../meshes/left_knee_link.dae
- link left_shoulder_pitch_link: geometry collision mesh filename=../meshes/left_shoulder_pitch_link.glb; visual mesh filename=../meshes/left_shoulder_pitch_link.dae
- link left_shoulder_roll_link: geometry collision mesh filename=../meshes/left_shoulder_roll_link.glb; visual mesh filename=../meshes/left_shoulder_roll_link.dae
- link left_shoulder_yaw_link: geometry collision mesh filename=../meshes/left_shoulder_yaw_link.glb; visual mesh filename=../meshes/left_shoulder_yaw_link.dae
- link pelvis: geometry collision mesh filename=../meshes/pelvis.glb; visual mesh filename=../meshes/pelvis.dae
- link right_ankle_link: geometry collision mesh filename=../meshes/right_ankle_link.glb; visual mesh filename=../meshes/right_ankle_link.dae
- link right_elbow_link: geometry collision mesh filename=../meshes/right_elbow_link.glb; visual mesh filename=../meshes/right_elbow_link.dae
- link right_hip_pitch_link: geometry collision mesh filename=../meshes/right_hip_pitch_link.glb; visual mesh filename=../meshes/right_hip_pitch_link.dae
- link right_hip_roll_link: geometry collision mesh filename=../meshes/right_hip_roll_link.glb; visual mesh filename=../meshes/right_hip_roll_link.dae
- link right_hip_yaw_link: geometry collision mesh filename=../meshes/right_hip_yaw_link.glb; visual mesh filename=../meshes/right_hip_yaw_link.dae
- link right_knee_link: geometry collision mesh filename=../meshes/right_knee_link.glb; visual mesh filename=../meshes/right_knee_link.dae
- link right_shoulder_pitch_link: geometry collision mesh filename=../meshes/right_shoulder_pitch_link.glb; visual mesh filename=../meshes/right_shoulder_pitch_link.dae
- link right_shoulder_roll_link: geometry collision mesh filename=../meshes/right_shoulder_roll_link.glb; visual mesh filename=../meshes/right_shoulder_roll_link.dae
- link right_shoulder_yaw_link: geometry collision mesh filename=../meshes/right_shoulder_yaw_link.glb; visual mesh filename=../meshes/right_shoulder_yaw_link.dae
Joints:
- removed joint d435_left_imager_joint
- removed joint d435_rgb_module_joint
- removed joint mid360_joint

Commit message: new envs, simplified contact version of h1 robot

File: mani_skill/assets/robots/unitree_h1/urdf/h1.urdf (robot description, URDF)
Before this commit: robot h1_description, 22 links, 21 joints
Links:
- link left_ankle_link: geometry collision mesh filename=../meshes/left_ankle_link.glb.coacd.ply; visual mesh filename=../meshes/left_ankle_link.dae
- link left_elbow_link: geometry collision mesh filename=../meshes/left_elbow_link.glb.coacd.ply; visual mesh filename=../meshes/left_elbow_link.dae
- link left_hip_pitch_link: geometry collision mesh filename=../meshes/left_hip_pitch_link.glb.coacd.ply; visual mesh filename=../meshes/left_hip_pitch_link.dae
- link left_hip_roll_link: geometry collision mesh filename=../meshes/left_hip_roll_link.glb.coacd.ply; visual mesh filename=../meshes/left_hip_roll_link.dae
- link left_hip_yaw_link: geometry collision mesh filename=../meshes/left_hip_yaw_link.glb.coacd.ply; visual mesh filename=../meshes/left_hip_yaw_link.dae
- link left_knee_link: geometry collision mesh filename=../meshes/left_knee_link.glb.coacd.ply; visual mesh filename=../meshes/left_knee_link.dae
- link left_shoulder_pitch_link: geometry collision mesh filename=../meshes/left_shoulder_pitch_link.glb.coacd.ply; visual mesh filename=../meshes/left_shoulder_pitch_link.dae
- link left_shoulder_roll_link: geometry collision mesh filename=../meshes/left_shoulder_roll_link.glb.coacd.ply; visual mesh filename=../meshes/left_shoulder_roll_link.dae
- link left_shoulder_yaw_link: geometry collision mesh filename=../meshes/left_shoulder_yaw_link.glb.coacd.ply; visual mesh filename=../meshes/left_shoulder_yaw_link.dae
- link pelvis: geometry collision mesh filename=../meshes/pelvis.glb.coacd.ply; visual mesh filename=../meshes/pelvis.dae
- link right_ankle_link: geometry collision mesh filename=../meshes/right_ankle_link.glb.coacd.ply; visual mesh filename=../meshes/right_ankle_link.dae
- link right_elbow_link: geometry collision mesh filename=../meshes/right_elbow_link.glb.coacd.ply; visual mesh filename=../meshes/right_elbow_link.dae
- link right_hip_pitch_link: geometry collision mesh filename=../meshes/right_hip_pitch_link.glb.coacd.ply; visual mesh filename=../meshes/right_hip_pitch_link.dae
- link right_hip_roll_link: geometry collision mesh filename=../meshes/right_hip_roll_link.glb.coacd.ply; visual mesh filename=../meshes/right_hip_roll_link.dae
- link right_hip_yaw_link: geometry collision mesh filename=../meshes/right_hip_yaw_link.glb.coacd.ply; visual mesh filename=../meshes/right_hip_yaw_link.dae
- link right_knee_link: geometry collision mesh filename=../meshes/right_knee_link.glb.coacd.ply; visual mesh filename=../meshes/right_knee_link.dae
- link right_shoulder_pitch_link: geometry collision mesh filename=../meshes/right_shoulder_pitch_link.glb.coacd.ply; visual mesh filename=../meshes/right_shoulder_pitch_link.dae
- link right_shoulder_roll_link: geometry collision mesh filename=../meshes/right_shoulder_roll_link.glb.coacd.ply; visual mesh filename=../meshes/right_shoulder_roll_link.dae
- link right_shoulder_yaw_link: geometry collision mesh filename=../meshes/right_shoulder_yaw_link.glb.coacd.ply; visual mesh filename=../meshes/right_shoulder_yaw_link.dae
- link torso_link: geometry collision mesh filename=../meshes/torso_link.glb.coacd.ply; visual mesh filename=../meshes/torso_link.dae
