Commit message: tune joint limits for easy rl

File: mani_skill/assets/robots/anymal-c/urdf/anymal_original.urdf (robot description, URDF)
Before this commit: robot anymal, 78 links, 77 joints
Joints:
- joint LF_HAA: limit lower=-0.51 upper=0.49 effort=80.0 velocity=7.5 -> lower=-0.72 upper=0.49 effort=80.0 velocity=7.5
- joint LF_HFE: limit lower=-0.1 upper=0.9 effort=80.0 velocity=7.5 -> lower=-9.42477796077 upper=9.42477796077 effort=80.0 velocity=7.5
- joint LF_KFE: limit lower=-1.3 upper=-0.3 effort=80.0 velocity=7.5 -> lower=-9.42477796077 upper=9.42477796077 effort=80.0 velocity=7.5
- joint LH_HAA: limit lower=-0.51 upper=0.49 effort=80.0 velocity=7.5 -> lower=-0.72 upper=0.49 effort=80.0 velocity=7.5
- joint LH_HFE: limit lower=-0.9 upper=0.1 effort=80.0 velocity=7.5 -> lower=-9.42477796077 upper=9.42477796077 effort=80.0 velocity=7.5
- joint LH_KFE: limit lower=0.3 upper=1.3 effort=80.0 velocity=7.5 -> lower=-9.42477796077 upper=9.42477796077 effort=80.0 velocity=7.5
- joint RF_HAA: limit lower=-0.49 upper=0.51 effort=80.0 velocity=7.5 -> lower=-0.49 upper=0.72 effort=80.0 velocity=7.5
- joint RF_HFE: limit lower=-0.1 upper=0.9 effort=80.0 velocity=7.5 -> lower=-9.42477796077 upper=9.42477796077 effort=80.0 velocity=7.5
- joint RF_KFE: limit lower=-1.3 upper=-0.3 effort=80.0 velocity=7.5 -> lower=-9.42477796077 upper=9.42477796077 effort=80.0 velocity=7.5
- joint RH_HAA: limit lower=-0.49 upper=0.51 effort=80.0 velocity=7.5 -> lower=-0.49 upper=0.72 effort=80.0 velocity=7.5
- joint RH_HFE: limit lower=-0.9 upper=0.1 effort=80.0 velocity=7.5 -> lower=-9.42477796077 upper=9.42477796077 effort=80.0 velocity=7.5
- joint RH_KFE: limit lower=0.3 upper=1.3 effort=80.0 velocity=7.5 -> lower=-9.42477796077 upper=9.42477796077 effort=80.0 velocity=7.5
