Commit message: Support xarm6 in TableSceneBuilder, fix xarm6 hand camera pose

File: mani_skill/assets/robots/xarm6/xarm6_xarmgripper.urdf (robot description, URDF)
Before this commit: robot xarm6, 17 links, 16 joints
Joints:
- joint eef_joint: origin xyz=0 0 0.15 rpy=0 0 0 -> xyz=0 0 0.172 rpy=0 0 0
