Commit message: Clean xarm6_allegro assets, add xarm6 SRDFs

File: mani_skill/assets/robots/xarm6/xarm6_allegro_right.urdf (robot description, URDF)
Before this commit: robot xarm6_allegro, 31 links, 30 joints
Links:
- link base_link: geometry collision box size=0.0414 0.0538 0.0428; collision box size=0.0414 0.0720 0.013
- link link_0.0: geometry collision box size=0.0196 0.0275 0.0164; visual mesh filename=../allegro/meshes/visual/link_0.0.glb
- link link_1.0: geometry collision box size=0.0196 0.0275 0.054; visual mesh filename=../allegro/meshes/visual/link_1.0.glb
- link link_10.0: geometry collision box size=0.0196 0.0275 0.0384; visual mesh filename=../allegro/meshes/visual/link_2.0.glb
- link link_11.0: geometry collision box size=0.0196 0.0269 0.022; visual mesh filename=../allegro/meshes/visual/link_3.0.glb
- link link_11.0_tip: geometry collision mesh filename=../allegro/meshes/collision/link_tip.obj; visual mesh filename=../allegro/meshes/visual/link_tip.glb
- link link_12.0: geometry collision box size=0.0358 0.034 0.0455; visual mesh filename=../allegro/meshes/visual/link_12.0_right.glb
- link link_13.0: geometry collision box size=0.0196 0.0275 0.0177; visual mesh filename=../allegro/meshes/visual/link_13.0.glb
- link link_14.0: geometry collision box size=0.0196 0.0275 0.0514; visual mesh filename=../allegro/meshes/visual/link_14.0.glb
- link link_15.0: geometry collision box size=0.0196 0.0269 0.04; visual mesh filename=../allegro/meshes/visual/link_15.0.glb
- link link_15.0_tip: geometry collision mesh filename=../allegro/meshes/collision/link_tip.obj; visual mesh filename=../allegro/meshes/visual/link_tip.glb
- link link_2.0: geometry collision box size=0.0196 0.0275 0.0384; visual mesh filename=../allegro/meshes/visual/link_2.0.glb
- link link_3.0: geometry collision box size=0.0196 0.0269 0.022; visual mesh filename=../allegro/meshes/visual/link_3.0.glb
- link link_3.0_tip: geometry collision mesh filename=../allegro/meshes/collision/link_tip.obj; visual mesh filename=../allegro/meshes/visual/link_tip.glb
- link link_4.0: geometry collision box size=0.0196 0.0275 0.0164; visual mesh filename=../allegro/meshes/visual/link_0.0.glb
- link link_5.0: geometry collision box size=0.0196 0.0275 0.054; visual mesh filename=../allegro/meshes/visual/link_1.0.glb
- link link_6.0: geometry collision box size=0.0196 0.0275 0.0384; visual mesh filename=../allegro/meshes/visual/link_2.0.glb
- link link_7.0: geometry collision box size=0.0196 0.0269 0.022; visual mesh filename=../allegro/meshes/visual/link_3.0.glb
- link link_7.0_tip: geometry collision mesh filename=../allegro/meshes/collision/link_tip.obj; visual mesh filename=../allegro/meshes/visual/link_tip.glb
- link link_8.0: geometry collision box size=0.0196 0.0275 0.0164; visual mesh filename=../allegro/meshes/visual/link_0.0.glb
- link link_9.0: geometry collision box size=0.0196 0.0275 0.054; visual mesh filename=../allegro/meshes/visual/link_1.0.glb
