Commit message: Fix PlaceCube reward and motionplanning demo generation for xarm6_pandagripper

File: mani_skill/assets/robots/xarm6/xarm6_pandagripper.urdf (robot description, URDF)
Before this commit: robot xarm6, 16 links, 15 joints
Joints:
- joint panda_finger_joint1: limit lower=0.0 upper=0.04 effort=100 velocity=0.2 -> lower=-0.04 upper=0.04 effort=100 velocity=0.2
- joint panda_finger_joint2: limit lower=0.0 upper=0.04 effort=100 velocity=0.2 -> lower=-0.04 upper=0.04 effort=100 velocity=0.2
