Commit message: fixes

File: mani_skill/assets/robots/g1_humanoid/g1_simplified_upper_body.urdf (robot description, URDF)
Before this commit: robot g1, 44 links, 43 joints
Links:
- link head_link: geometry collision mesh filename=meshes/head_link.STL; visual mesh filename=meshes/head_link.STL

Commit message: work

File: mani_skill/assets/robots/g1_humanoid/g1_simplified_upper_body.urdf (robot description, URDF)
Before this commit: robot g1, 44 links, 43 joints
Links:
- added link left_tcp_link; visual sphere radius=0.012
- added link right_tcp_link; visual sphere radius=0.012
Joints:
- added joint left_tcp_joint: type fixed, parent left_palm_link, child left_tcp_link, origin xyz=0 0 0 rpy=0 0 0, axis 0 0 0
- added joint right_tcp_joint: type fixed, parent right_palm_link, child right_tcp_link, origin xyz=0 0 0 rpy=0 0 0, axis 0 0 0

Commit message: fix tcp poses

File: mani_skill/assets/robots/g1_humanoid/g1_simplified_upper_body.urdf (robot description, URDF)
Before this commit: robot g1, 46 links, 45 joints
Joints:
- joint left_tcp_joint: origin xyz=0 0 0 rpy=0 0 0 -> xyz=0.07 -0.035 0 rpy=0 0 0
- joint right_tcp_joint: origin xyz=0 0 0 rpy=0 0 0 -> xyz=0.07 0.035 0 rpy=0 0 0

Commit message: work

File: mani_skill/assets/robots/g1_humanoid/g1_simplified_upper_body.urdf (robot description, URDF)
Before this commit: robot g1, 46 links, 45 joints
Links:
- link left_tcp_link: geometry 
- link right_tcp_link: geometry 
