Commit message: lower case files, srdf and simplified urdfs added with fixed gripper collisions.

File: mani_skill/assets/robots/koch/follower_arm_v1.1_simplified.urdf (robot description, URDF)
Before this commit: robot koch, 8 links, 7 joints
Links:
- added link gripper_tcp
- link base_link: geometry visual mesh filename=package://koch/meshes/base_link.stl
Joints:
- added joint gripper_tcp_joint: type fixed, parent link_6, child gripper_tcp, origin xyz=-0.008 0 -0.065 rpy=0 0 0

Commit message: remodelled assets to be more realistic, simplified urdfs, customizable robot colors

File: mani_skill/assets/robots/koch/follower_arm_v1.1_simplified.urdf (robot description, URDF)
Before this commit: robot koch, 9 links, 8 joints
Links:
- link base_link: geometry visual mesh filename=package://koch/meshes/base_link.glb
- link gripper: geometry collision mesh filename=package://koch/meshes/gripper.stl; visual mesh filename=package://koch/meshes/gripper.glb
- link link_1: geometry collision mesh filename=package://koch/meshes/link_1.stl; visual mesh filename=package://koch/meshes/link_1_motor.glb
- link link_2: geometry visual mesh filename=package://koch/meshes/link_2_motor.glb; visual mesh filename=package://koch/meshes/link_2_rotation_connector.glb
- link link_3: geometry collision mesh filename=package://koch/meshes/link_3.stl; visual mesh filename=package://koch/meshes/link_3_motor.glb
- link link_4: geometry collision mesh filename=package://koch/meshes/link_4.stl; visual mesh filename=package://koch/meshes/link_4_motor.glb
- link link_5: geometry collision mesh filename=package://koch/meshes/link_5.stl; visual mesh filename=package://koch/meshes/link_5_motor.glb
- link link_6: geometry collision mesh filename=package://koch/meshes/link_6.stl; visual mesh filename=package://koch/meshes/link_6_motor.glb
Joints:
- joint joint_2: limit lower=-3.14159 upper=3.14159 -> lower=-1.4 upper=1.5707
- joint joint_3: limit lower=-3.14159 upper=3.14159 -> lower=-1.5707 upper=1.3
- joint joint_4: limit lower=-3.14159 upper=3.14159 -> lower=-3.14159 upper=0.5

Commit message: modelled collision meshes

File: mani_skill/assets/robots/koch/follower_arm_v1.1_simplified.urdf (robot description, URDF)
Before this commit: robot koch, 9 links, 8 joints
Links:
- link gripper: geometry collision mesh filename=package://koch/meshes/gripper_collision_part_1.glb; collision mesh filename=package://koch/meshes/gripper_collision_part_2.glb
- link link_6: geometry collision box size=0.011 0.0295 0.0344; collision mesh filename=package://koch/meshes/link_6_collision_part_2.glb

Commit message: matched qpos zero vector to real robot, limits estimated until real robot comes in

File: mani_skill/assets/robots/koch/follower_arm_v1.1_simplified.urdf (robot description, URDF)
Before this commit: robot koch, 9 links, 8 joints
Joints:
- joint joint_2: limit lower=-1.4 upper=1.5707 -> lower=-2.5 upper=0; origin xyz=0.020713 0 0.015368 rpy=0 0 0 -> xyz=0.020713 0 0.015368 rpy=1.5707963 0 0
- joint joint_3: limit lower=-1.5707 upper=1.3 -> lower=0 upper=3.04; origin xyz=-0.038026 -0.014951  0.108424 rpy=0 0 0 -> xyz=-0.038026 -0.014951  0.108424 rpy=-1.5707963 0 0
- joint joint_4: limit lower=-3.14159 upper=0.5 -> lower=-1 upper=2.14159; origin xyz=-0.000251 -0.100502  0.002641 rpy=0 0 0 -> xyz=-0.000251 -0.100502  0.002641 rpy=-1.5707963 0 0
- joint joint_5: origin xyz=0.019234  0.00037 -0.044779 rpy=0 0 0 -> xyz=0.019234  0.00037 -0.044779 rpy=0 0 -1.5707963

Commit message: added custom convex glb collisions for links 2,3,4

File: mani_skill/assets/robots/koch/follower_arm_v1.1_simplified.urdf (robot description, URDF)
Before this commit: robot koch, 9 links, 8 joints
Links:
- link link_2: geometry collision mesh filename=package://koch/meshes/link_2_collision_chassis.glb; collision mesh filename=package://koch/meshes/link_2_collision_motor.glb
- link link_3: geometry collision mesh filename=package://koch/meshes/link_3_collision_chassis_part_1.glb; collision mesh filename=package://koch/meshes/link_3_collision_chassis_part_2.glb
- link link_4: geometry collision mesh filename=package://koch/meshes/link_4_collision_chassis_part_1.glb; collision mesh filename=package://koch/meshes/link_4_collision_chassis_part_2.glb
Joints:
- joint joint_3: limit lower=0 upper=3.04 -> lower=0 upper=3.05

Commit message: Update follower_arm_v1.1_simplified.urdf

File: mani_skill/assets/robots/koch/follower_arm_v1.1_simplified.urdf (robot description, URDF)
Before this commit: robot koch, 9 links, 8 joints
Joints:
- joint joint_1: axis 0 0 1 -> 0 0 -1
- joint joint_2: axis 1 0 0 -> -1 0 0; limit lower=-2.5 upper=0 -> lower=0 upper=2.5
- joint joint_6: axis 0 1 0 -> 0 -1 0; limit lower=-1.75 upper=0 -> lower=0 upper=1.75

Commit message: lerobot dataset reader and transfer of simpler-env sysid implementation from ms2 to ms3, with added qpos_mse objective

File: mani_skill/assets/robots/koch/follower_arm_v1.1_simplified.urdf (robot description, URDF)
Before this commit: robot koch, 9 links, 8 joints
Joints:
- joint joint_5: axis 0 0 1 -> 0 0 -1

Commit message: cube size and friction DR grab_cube env

File: mani_skill/assets/robots/koch/follower_arm_v1.1_simplified.urdf (robot description, URDF)
Before this commit: robot koch, 9 links, 8 joints
Links:
- added link gripper_tcp2
Joints:
- added joint gripper_tcp_joint2: type fixed, parent gripper, child gripper_tcp2, origin xyz=-0.0135 0.0172 -0.0514 rpy=0 0 0

Commit message: grab cube reward shaped

File: mani_skill/assets/robots/koch/follower_arm_v1.1_simplified.urdf (robot description, URDF)
Before this commit: robot koch, 9 links, 8 joints
Links:
- added link gripper_tcp2
Joints:
- added joint gripper_tcp_joint2: type fixed, parent gripper, child gripper_tcp2, origin xyz=-0.010505 0.017151 -0.041535 rpy=0 0 0
- joint gripper_tcp_joint: origin xyz=-0.008 0 -0.065 rpy=0 0 0 -> xyz=-0.011337 0 -0.05574 rpy=0 0 0

Commit message: allows BaseDigitalTwinEnv to render the overlay images during evaluation in ppo, grab_cube environment and koch robot controller updated with target controller which is more compatible with real robot, and joint actions are greatly limited resulting in a smoother policy and safer robot, koch follower arm qpos ranges updated for a safer robot

File: mani_skill/assets/robots/koch/follower_arm_v1.1_simplified.urdf (robot description, URDF)
Before this commit: robot koch, 10 links, 9 joints
Joints:
- joint joint_2: limit lower=0 upper=2.5 -> lower=0 upper=2.2

Commit message: sim2real pipeline updated, organization, rewards, RealBaseEnv and RealBaseAgent, extended by MS3Koch to mimic simulation koch and simulation environments - reuses sim controller

File: mani_skill/assets/robots/koch/follower_arm_v1.1_simplified.urdf (robot description, URDF)
Before this commit: robot koch, 10 links, 9 joints
Links:
- added link back_tcp
- link base_link: geometry visual mesh filename=package://koch/meshes/centered_base_link.stl
Joints:
- added joint back_tcp_joint: type fixed, parent link_6, child back_tcp, origin xyz=-0.00 0 -0.023 rpy=0 0 0
- joint fixed_joint: origin xyz=0.005766 -0.028665  0.018513 rpy=0 0 0 -> xyz=0.0005 -0.056 0.021 rpy=0 0 0
- joint gripper_tcp_joint: origin xyz=-0.011337 0 -0.05574 rpy=0 0 0 -> xyz=-0.008 0 -0.065 rpy=0 0 0
- joint gripper_tcp_joint2: origin xyz=-0.010505 0.017151 -0.041535 rpy=0 0 0 -> xyz=-0.0135 0.0172 -0.0514 rpy=0 0 0
- joint joint_4: limit lower=-1 upper=2.14159 -> lower=-1.5 upper=2.14159
- joint joint_6: limit lower=0 upper=1.75 -> lower=0 upper=1.6
