Commit message: work

File: mani_skill/assets/robots/koch/follower_arm_v1.1.urdf (robot description, URDF)
Before this commit: robot koch, 9 links, 8 joints
Links:
- added link back_tcp
- added link gripper_tcp2
- link base_link: geometry visual mesh filename=package://koch/meshes/centered_base_link.stl
- link gripper: geometry collision mesh filename=package://koch/meshes/gripper_collision_part_1.glb; collision mesh filename=package://koch/meshes/gripper_collision_part_2.glb
- link link_1: geometry collision mesh filename=package://koch/meshes/link_1.stl; visual mesh filename=package://koch/meshes/link_1_motor.glb
- link link_2: geometry collision mesh filename=package://koch/meshes/link_2_collision_chassis.glb; collision mesh filename=package://koch/meshes/link_2_collision_motor.glb
- link link_3: geometry collision mesh filename=package://koch/meshes/link_3_collision_chassis_part_1.glb; collision mesh filename=package://koch/meshes/link_3_collision_chassis_part_2.glb
- link link_4: geometry collision mesh filename=package://koch/meshes/link_4_collision_chassis_part_1.glb; collision mesh filename=package://koch/meshes/link_4_collision_chassis_part_2.glb
- link link_5: geometry collision mesh filename=package://koch/meshes/link_5.stl; visual mesh filename=package://koch/meshes/link_5_motor.glb
- link link_6: geometry collision box size=0.011 0.0295 0.0344; collision mesh filename=package://koch/meshes/link_6_collision_part_2.glb
Joints:
- added joint back_tcp_joint: type fixed, parent link_6, child back_tcp, origin xyz=-0.00 0 -0.023 rpy=0 0 0
- added joint gripper_tcp_joint2: type fixed, parent gripper, child gripper_tcp2, origin xyz=-0.0135 0.0172 -0.0514 rpy=0 0 0
- joint fixed_joint: origin xyz=0.005766 -0.028665  0.018513 rpy=0 0 0 -> xyz=0.0005 -0.056 0.021 rpy=0 0 0
- joint joint_1: axis 0 0 1 -> 0 0 -1
- joint joint_2: axis 1 0 0 -> -1 0 0; limit lower=-3.14159 upper=3.14159 -> lower=0 upper=2.2; origin xyz=0.020713 0 0.015368 rpy=0 0 0 -> xyz=0.020713 0 0.015368 rpy=1.5707963 0 0
- joint joint_3: limit lower=-3.14159 upper=3.14159 -> lower=0 upper=3.05; origin xyz=-0.038026 -0.014951  0.108424 rpy=0 0 0 -> xyz=-0.038026 -0.014951  0.108424 rpy=-1.5707963 0 0
- joint joint_4: limit lower=-3.14159 upper=3.14159 -> lower=-1.5 upper=2.14159; origin xyz=-0.000251 -0.100502  0.002641 rpy=0 0 0 -> xyz=-0.000251 -0.100502  0.002641 rpy=-1.5707963 0 0
- joint joint_5: axis 0 0 1 -> 0 0 -1; origin xyz=0.019234  0.00037 -0.044779 rpy=0 0 0 -> xyz=0.019234  0.00037 -0.044779 rpy=0 0 -1.5707963
- joint joint_6: axis 0 1 0 -> 0 -1 0; limit lower=-1.75 upper=0 -> lower=0 upper=1.6
