Commit message: modelling

File: mani_skill/assets/robots/inspire_hand/urdf/end_effector/inspire_hand/inspire_hand_left.urdf (robot description, URDF)
Before this commit: robot inspire_hand, 20 links, 19 joints
Joints:
- joint left_hand_index_PIP_joint: mimic joint=left_hand_index_MCP_joint multiplier=1.06399 offset=-0.16734800000000002 -> (none)
- joint left_hand_middle_PIP_joint: mimic joint=left_hand_middle_MCP_joint multiplier=1.06399 offset=-0.16734800000000002 -> (none)
- joint left_hand_pinky_PIP_joint: mimic joint=left_hand_pinky_MCP_joint multiplier=1.06399 offset=-0.16734800000000002 -> (none)
- joint left_hand_ring_PIP_joint: mimic joint=left_hand_ring_MCP_joint multiplier=1.06399 offset=-0.16734800000000002 -> (none)
- joint left_hand_thumb_IP_joint: mimic joint=left_hand_thumb_CMC_pitch_joint multiplier=0.6666666666666667 offset=-0.040724349213201026 -> (none)
- joint left_hand_thumb_MCP_joint: mimic joint=left_hand_thumb_CMC_pitch_joint multiplier=1.3333333333333335 offset=-0.08144869842640205 -> (none)

File: mani_skill/assets/robots/inspire_hand/urdf/end_effector/inspire_hand/inspire_hand_right_floating.urdf (robot description, URDF)
Before this commit: robot inspire_hand, 26 links, 25 joints
Links:
- removed link root
- removed link root_arm_1_link_1
- removed link root_arm_1_link_2
- removed link root_arm_1_link_3
- removed link root_arm_1_link_4
- removed link root_arm_1_link_5
Joints:
- removed joint root_x_axis_joint
- removed joint root_x_rot_joint
- removed joint root_y_axis_joint
- removed joint root_y_rot_joint
- removed joint root_z_axis_joint
- removed joint root_z_rot_joint
