Commit message: modelling

File: mani_skill/assets/robots/inspire_hand/urdf/end_effector/inspire_hand/inspire_hand_right_floating.urdf (robot description, URDF)
Before this commit: robot inspire_hand, 20 links, 19 joints
Links:
- added link root, mass 0
- added link root_arm_1_link_1, mass 0
- added link root_arm_1_link_2, mass 0
- added link root_arm_1_link_3, mass 0
- added link root_arm_1_link_4, mass 0
- added link root_arm_1_link_5, mass 0
Joints:
- added joint root_x_axis_joint: type prismatic, parent root, child root_arm_1_link_1, axis 1 0 0, limit lower=-20 upper=20 effort=100 velocity=0.50
- added joint root_x_rot_joint: type revolute, parent root_arm_1_link_3, child root_arm_1_link_4, axis 1 0 0, limit lower=-20 upper=20 effort=100 velocity=0.50
- added joint root_y_axis_joint: type prismatic, parent root_arm_1_link_1, child root_arm_1_link_2, axis 0 1 0, limit lower=-20 upper=20 effort=100 velocity=0.50
- added joint root_y_rot_joint: type revolute, parent root_arm_1_link_4, child root_arm_1_link_5, axis 0 1 0, limit lower=-20 upper=20 effort=100 velocity=0.50
- added joint root_z_axis_joint: type prismatic, parent root_arm_1_link_2, child root_arm_1_link_3, axis 0 0 1, limit lower=-20 upper=20 effort=100 velocity=0.50
- added joint root_z_rot_joint: type revolute, parent root_arm_1_link_5, child right_hand_wrist_base_link, axis 0 0 1, limit lower=-20 upper=20 effort=100 velocity=0.50

Commit message: work

File: mani_skill/assets/robots/inspire_hand/urdf/end_effector/inspire_hand/inspire_hand_right_floating.urdf (robot description, URDF)
Before this commit: robot inspire_hand, 26 links, 25 joints
Links:
- removed link root
- removed link root_arm_1_link_1
- removed link root_arm_1_link_2
- removed link root_arm_1_link_3
- removed link root_arm_1_link_4
- removed link root_arm_1_link_5
Joints:
- removed joint root_x_axis_joint
- removed joint root_x_rot_joint
- removed joint root_y_axis_joint
- removed joint root_y_rot_joint
- removed joint root_z_axis_joint
- removed joint root_z_rot_joint
- joint right_hand_index_PIP_joint: mimic (none) -> joint=right_hand_index_MCP_joint multiplier=1.06399 offset=-0.16734800000000002
- joint right_hand_middle_PIP_joint: mimic (none) -> joint=right_hand_middle_MCP_joint multiplier=1.06399 offset=-0.16734800000000002
- joint right_hand_pinky_PIP_joint: mimic (none) -> joint=right_hand_pinky_MCP_joint multiplier=1.06399 offset=-0.16734800000000002
- joint right_hand_ring_PIP_joint: mimic (none) -> joint=right_hand_ring_MCP_joint multiplier=1.06399 offset=-0.16734800000000002
- joint right_hand_thumb_IP_joint: mimic (none) -> joint=right_hand_thumb_CMC_pitch_joint multiplier=0.6666666666666667 offset=-0.040724349213201026
- joint right_hand_thumb_MCP_joint: mimic (none) -> joint=right_hand_thumb_CMC_pitch_joint multiplier=1.3333333333333335 offset=-0.08144869842640205

Commit message: more stable

File: mani_skill/assets/robots/inspire_hand/urdf/end_effector/inspire_hand/inspire_hand_right_floating.urdf (robot description, URDF)
Before this commit: robot inspire_hand, 20 links, 19 joints
Links:
- added link root, mass 0
- added link root_arm_1_link_1, mass 0
- added link root_arm_1_link_2, mass 0
- added link root_arm_1_link_3, mass 0
- added link root_arm_1_link_4, mass 0
- added link root_arm_1_link_5, mass 0
Joints:
- added joint root_x_axis_joint: type prismatic, parent root, child root_arm_1_link_1, axis 1 0 0, limit lower=-20 upper=20 effort=100 velocity=0.50
- added joint root_x_rot_joint: type revolute, parent root_arm_1_link_3, child root_arm_1_link_4, axis 1 0 0, limit lower=-20 upper=20 effort=100 velocity=0.50
- added joint root_y_axis_joint: type prismatic, parent root_arm_1_link_1, child root_arm_1_link_2, axis 0 1 0, limit lower=-20 upper=20 effort=100 velocity=0.50
- added joint root_y_rot_joint: type revolute, parent root_arm_1_link_4, child root_arm_1_link_5, axis 0 1 0, limit lower=-20 upper=20 effort=100 velocity=0.50
- added joint root_z_axis_joint: type prismatic, parent root_arm_1_link_2, child root_arm_1_link_3, axis 0 0 1, limit lower=-20 upper=20 effort=100 velocity=0.50
- added joint root_z_rot_joint: type revolute, parent root_arm_1_link_5, child right_hand_wrist_base_link, axis 0 0 1, limit lower=-20 upper=20 effort=100 velocity=0.50
- joint right_hand_index_PIP_joint: limit lower=-1.56 upper=0.04545 effort=1 velocity=0.5 -> lower=-1.5930946000000001 upper=0.04545 effort=1 velocity=0.5
- joint right_hand_middle_PIP_joint: limit lower=-1.56 upper=0.04545 effort=1 velocity=0.5 -> lower=-1.5930946000000001 upper=0.04545 effort=1 velocity=0.5
- joint right_hand_pinky_PIP_joint: limit lower=-1.56 upper=0.04545 effort=1 velocity=0.5 -> lower=-1.5930946000000001 upper=0.04545 effort=1 velocity=0.5
- joint right_hand_ring_PIP_joint: limit lower=-1.56 upper=0.04545 effort=1 velocity=0.5 -> lower=-1.5930946000000001 upper=0.04545 effort=1 velocity=0.5
- joint right_hand_thumb_IP_joint: mimic joint=right_hand_thumb_CMC_pitch_joint multiplier=0.6666666666666667 offset=-0.040724349213201026 -> joint=right_hand_thumb_MCP_joint multiplier=0.888 offset=0
