Commit message: fix urdf

File: mani_skill/assets/robots/so100/SO_5DOF_ARM100_8j/original.urdf (robot description, URDF)
Before this commit: robot SO_5DOF_ARM100_8j_URDF.SLDASM, 7 links, 6 joints
Joints:
- joint Elbow: limit (none) -> lower=-0.2 upper=3.14159 effort=0 velocity=0; origin xyz=0 0.11257 0.028 rpy=0 0 0 -> xyz=0 0.11257 0.028 rpy=-1.5708 0 0; type continuous -> revolute
- joint Jaw: limit (none) -> lower=0 upper=1.7 effort=0 velocity=0; origin xyz=-0.0202 -0.0244 0 rpy=3.1416 0 3.1416 -> xyz=-0.0202 -0.0244 0 rpy=3.1416 0 3.33; type continuous -> revolute
- joint Pitch: limit lower=0 upper=3.45 effort=0 velocity=0 -> lower=-0.1 upper=3.45 effort=0 velocity=0; origin xyz=0 0.1025 0.0306 rpy=0 0 0 -> xyz=0 0.1025 0.0306 rpy=1.5708 0 0
- joint Wrist_Pitch: limit (none) -> lower=-1.8 upper=1.8 effort=0 velocity=0; origin xyz=0 0.0052 0.1349 rpy=0 0 0 -> xyz=0 0.0052 0.1349 rpy=-1.5708 0 0; type continuous -> revolute
- joint Wrist_Roll: limit (none) -> lower=-3.14159 upper=3.14159 effort=0 velocity=0; origin xyz=0 -0.0601 0 rpy=0 0 0 -> xyz=0 -0.0601 0 rpy=0 -1.5708 0; type continuous -> revolute

Commit message: fix collision meshes and reset controller in robot demo code

File: mani_skill/assets/robots/so100/SO_5DOF_ARM100_8j/original.urdf (robot description, URDF)
Before this commit: robot SO_5DOF_ARM100_8j_URDF.SLDASM, 7 links, 6 joints
Links:
- link Fixed_Jaw: geometry collision mesh filename=meshes/Fixed_Jaw_part1.ply; collision mesh filename=meshes/Fixed_Jaw_part2.ply
- link Moving Jaw: geometry collision mesh filename=meshes/Moving_Jaw_part1.ply; collision mesh filename=meshes/Moving_Jaw_part2.ply

Commit message: fix urdf

File: mani_skill/assets/robots/so100/SO_5DOF_ARM100_8j/original.urdf (robot description, URDF)
Before this commit: robot SO_5DOF_ARM100_8j_URDF.SLDASM, 7 links, 6 joints
Joints:
- joint Wrist_Roll: axis 0 1 0 -> 0 -1 0; origin xyz=0 -0.0601 0 rpy=0 -1.5708 0 -> xyz=0 -0.0601 0 rpy=0 1.5708 0

Commit message: work

File: mani_skill/assets/robots/so100/SO_5DOF_ARM100_8j/original.urdf (robot description, URDF)
Before this commit: robot SO_5DOF_ARM100_8j_URDF.SLDASM, 7 links, 6 joints
Links:
- removed link Moving Jaw
- added link Moving_Jaw, mass 0.0202443794940372; collision mesh filename=meshes/Moving_Jaw_part1.ply; collision mesh filename=meshes/Moving_Jaw_part2.ply
Joints:
- joint Jaw: child Moving Jaw -> Moving_Jaw

Commit message: work

File: mani_skill/assets/robots/so100/SO_5DOF_ARM100_8j/original.urdf (robot description, URDF)
Before this commit: robot SO_5DOF_ARM100_8j_URDF.SLDASM, 7 links, 6 joints
Links:
- added link Fixed_Jaw_tip
- added link Moving_Jaw_tip
Joints:
- added joint Fixed_Jaw_tip_joint: type fixed, parent Fixed_Jaw, child Fixed_Jaw_tip, origin xyz=0.01 -0.097 0 rpy=0 0 0
- added joint Moving_Jaw_tip_joint: type fixed, parent Moving_Jaw, child Moving_Jaw_tip, origin xyz=-0.01 -0.073 0 rpy=0 0 0

Commit message: fixed so100 modelling

File: mani_skill/assets/robots/so100/SO_5DOF_ARM100_8j/original.urdf (robot description, URDF)
Before this commit: robot SO_5DOF_ARM100_8j_URDF.SLDASM, 7 links, 6 joints
Links:
- removed link Moving Jaw
- added link Fixed_Jaw_tip
- added link Moving_Jaw, mass 0.0202443794940372; collision mesh filename=meshes/Moving_Jaw_part1.ply; collision mesh filename=meshes/Moving_Jaw_part2.ply
- added link Moving_Jaw_tip
Joints:
- added joint Fixed_Jaw_tip_joint: type fixed, parent Fixed_Jaw, child Fixed_Jaw_tip, origin xyz=0.01 -0.097 0 rpy=0 0 0
- added joint Moving_Jaw_tip_joint: type fixed, parent Moving_Jaw, child Moving_Jaw_tip, origin xyz=-0.01 -0.073 0 rpy=0 0 0
- joint Jaw: child Moving Jaw -> Moving_Jaw

Commit message: better modelling

File: mani_skill/assets/robots/so100/SO_5DOF_ARM100_8j/original.urdf (robot description, URDF)
Before this commit: robot SO_5DOF_ARM100_8j_URDF.SLDASM, 9 links, 8 joints
Links:
- link Base: geometry collision mesh filename=meshes/base_link.glb; visual mesh filename=meshes/base_link.glb
- link Fixed_Jaw: geometry collision mesh filename=meshes/Fixed_Jaw_part1.ply; collision mesh filename=meshes/Fixed_Jaw_part2.ply
- link Lower_Arm: geometry collision mesh filename=meshes/lower_arm.glb; collision mesh filename=meshes/lower_arm_motor.glb
- link Rotation_Pitch: geometry collision mesh filename=meshes/rotation_pitch.glb; collision mesh filename=meshes/rotation_pitch_motor.glb
- link Upper_Arm: geometry collision mesh filename=meshes/upper_arm.glb; collision mesh filename=meshes/upper_arm_motor.glb
- link Wrist_Pitch_Roll: geometry collision mesh filename=meshes/wrist_pitch_roll.glb; collision mesh filename=meshes/wrist_pitch_roll_motor.glb
