Commit message: work

File: mani_skill/assets/robots/so100/SO_5DOF_ARM100_8j/so100.urdf (robot description, URDF)
Before this commit: robot SO_5DOF_ARM100_8j_URDF.SLDASM, 9 links, 8 joints
Links:
- link Base: geometry collision mesh filename=meshes/Base.stl; collision mesh filename=meshes/Base_Motor.stl
- link Fixed_Jaw: geometry collision mesh filename=meshes/Fixed_Jaw_part1.ply; collision mesh filename=meshes/Fixed_Jaw_part2.ply
- link Lower_Arm: geometry collision mesh filename=meshes/Lower_Arm.stl; collision mesh filename=meshes/Lower_Arm_Motor.stl
- link Moving_Jaw: geometry collision mesh filename=meshes/Moving_Jaw_part1.ply; collision mesh filename=meshes/Moving_Jaw_part2.ply
- link Rotation_Pitch: geometry collision mesh filename=meshes/Rotation_Pitch.stl; collision mesh filename=meshes/Rotation_Pitch_Motor.stl
- link Upper_Arm: geometry collision mesh filename=meshes/Upper_Arm.stl; collision mesh filename=meshes/Upper_Arm_Motor.stl
- link Wrist_Pitch_Roll: geometry collision mesh filename=meshes/Wrist_Pitch_Roll.stl; collision mesh filename=meshes/Wrist_Pitch_Roll_Motor.stl

Commit message: update so100 modelling to match the new lerobot system's modelling as well as joint namings

File: mani_skill/assets/robots/so100/SO_5DOF_ARM100_8j/so100.urdf (robot description, URDF)
Before this commit: robot SO_5DOF_ARM100_8j_URDF.SLDASM, 9 links, 8 joints
Joints:
- removed joint Elbow
- removed joint Pitch
- removed joint Rotation
- removed joint Wrist_Pitch
- removed joint Wrist_Roll
- added joint elbow_flex: type revolute, parent Upper_Arm, child Lower_Arm, origin xyz=0 0.11257 0.028 rpy=0 0 0, axis 1 0 0, limit lower=-1.5708 upper=1.5708 effort=0 velocity=0
- added joint shoulder_lift: type revolute, parent Rotation_Pitch, child Upper_Arm, origin xyz=0 0.1025 0.0306 rpy=0 0 0, axis 1 0 0, limit lower=-1.5708 upper=1.5708 effort=0 velocity=0
- added joint shoulder_pan: type revolute, parent Base, child Rotation_Pitch, origin xyz=0 -0.0452 0.0165 rpy=1.5708 0 0, axis 0 -1 0, limit lower=-2.0 upper=2.0 effort=0 velocity=0
- added joint wrist_flex: type revolute, parent Lower_Arm, child Wrist_Pitch_Roll, origin xyz=0 0.0052 0.1349 rpy=-1.5708 0 0, axis 1 0 0, limit lower=-1.8 upper=1.8 effort=0 velocity=0
- added joint wrist_roll: type revolute, parent Wrist_Pitch_Roll, child Fixed_Jaw, origin xyz=0 -0.0601 0 rpy=0 1.5708 0, axis 0 1 0, limit lower=-3.14159 upper=3.14159 effort=0 velocity=0

Commit message: fixes

File: mani_skill/assets/robots/so100/SO_5DOF_ARM100_8j/so100.urdf (robot description, URDF)
Before this commit: robot SO_5DOF_ARM100_8j_URDF.SLDASM, 9 links, 8 joints
Joints:
- removed joint Jaw
- added joint gripper: type revolute, parent Fixed_Jaw, child Moving_Jaw, origin xyz=-0.0202 -0.0244 0 rpy=0 3.14159 -0.9, axis 0 0 1, limit lower=-1.1 upper=1.1 effort=0 velocity=0

Commit message: SO100 modelling based on new lerobot hardware API and improved task design, and experimental cached reset method (#1125)
* work

* work

* Update grasp_cube.py

* tune

* work

* work

* w

* w

* fixes

* Update grasp_cube.py

* Update scratch.sh

* work

* fix camera poses not updating

* work

* fixes

* update so100 modelling to match the new lerobot system's modelling as well as joint namings

* fixes

* Update manipulator.py

* fixes

* fixes

* w

* Update so_100.py

* work

* w

* work

* w

* reverts

File: mani_skill/assets/robots/so100/SO_5DOF_ARM100_8j/so100.urdf (robot description, URDF)
Before this commit: robot SO_5DOF_ARM100_8j_URDF.SLDASM, 9 links, 8 joints
Joints:
- removed joint Elbow
- removed joint Jaw
- removed joint Pitch
- removed joint Rotation
- removed joint Wrist_Pitch
- removed joint Wrist_Roll
- added joint elbow_flex: type revolute, parent Upper_Arm, child Lower_Arm, origin xyz=0 0.11257 0.028 rpy=0 0 0, axis 1 0 0, limit lower=-1.5708 upper=1.5708 effort=0 velocity=0
- added joint gripper: type revolute, parent Fixed_Jaw, child Moving_Jaw, origin xyz=-0.0202 -0.0244 0 rpy=0 3.14159 -0.9, axis 0 0 1, limit lower=-1.1 upper=1.1 effort=0 velocity=0
- added joint shoulder_lift: type revolute, parent Rotation_Pitch, child Upper_Arm, origin xyz=0 0.1025 0.0306 rpy=0 0 0, axis 1 0 0, limit lower=-1.5708 upper=1.5708 effort=0 velocity=0
- added joint shoulder_pan: type revolute, parent Base, child Rotation_Pitch, origin xyz=0 -0.0452 0.0165 rpy=1.5708 0 0, axis 0 -1 0, limit lower=-2.0 upper=2.0 effort=0 velocity=0
- added joint wrist_flex: type revolute, parent Lower_Arm, child Wrist_Pitch_Roll, origin xyz=0 0.0052 0.1349 rpy=-1.5708 0 0, axis 1 0 0, limit lower=-1.8 upper=1.8 effort=0 velocity=0
- added joint wrist_roll: type revolute, parent Wrist_Pitch_Roll, child Fixed_Jaw, origin xyz=0 -0.0601 0 rpy=0 1.5708 0, axis 0 1 0, limit lower=-3.14159 upper=3.14159 effort=0 velocity=0
