Commit message: Fix: fetch pd_ee_target_delta_pose by using torso link as root for ik

File: mani_skill/assets/robots/fetch/fetch_torso_up.urdf (robot description, URDF)
Before this commit: robot fetch, 26 links, 25 joints
Links:
- removed link base_link
- removed link estop_link
- removed link l_wheel_link
- removed link laser_link
- removed link r_wheel_link
- removed link torso_fixed_link
Joints:
- removed joint estop_joint
- removed joint l_wheel_joint
- removed joint laser_joint
- removed joint r_wheel_joint
- removed joint torso_fixed_joint
- removed joint torso_lift_joint
