Commit message: work

File: mani_skill/assets/robots/inspire_hand/RH56DFX-2LR/urdf/inspire_hand_right_floating.urdf (robot description, URDF)
Before this commit: robot inspire_hand, 26 links, 25 joints
Links:
- link right_hand_hand_base_link: geometry collision mesh filename=../meshes/end_effector/inspire_hand/visual/R_hand_base_link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; visual mesh filename=../meshes/end_effector/inspire_hand/visual/R_hand_base_link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
- link right_hand_index_middle: geometry collision mesh filename=../meshes/end_effector/inspire_hand/visual/index_ring_middl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; visual mesh filename=../meshes/end_effector/inspire_hand/visual/index_ring_middl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
- link right_hand_index_proximal: geometry collision mesh filename=../meshes/end_effector/inspire_hand/visual/index_ring_proxi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; visual mesh filename=../meshes/end_effector/inspire_hand/visual/index_ring_proxi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
- link right_hand_middle_middle: geometry collision mesh filename=../meshes/end_effector/inspire_hand/visual/middle_middle.glb; visual mesh filename=../meshes/end_effector/inspire_hand/visual/middle_middle.glb
- link right_hand_middle_proximal: geometry collision mesh filename=../meshes/end_effector/inspire_hand/visual/middle_pinky_pro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; visual mesh filename=../meshes/end_effector/inspire_hand/visual/middle_pinky_pro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
- link right_hand_pinky_middle: geometry collision mesh filename=../meshes/end_effector/inspire_hand/visual/pinky_middle.glb; visual mesh filename=../meshes/end_effector/inspire_hand/visual/pinky_middle.glb
- link right_hand_pinky_proximal: geometry collision mesh filename=../meshes/end_effector/inspire_hand/visual/middle_pinky_pro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; visual mesh filename=../meshes/end_effector/inspire_hand/visual/middle_pinky_pro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
- link right_hand_ring_middle: geometry collision mesh filename=../meshes/end_effector/inspire_hand/visual/index_ring_middl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; visual mesh filename=../meshes/end_effector/inspire_hand/visual/index_ring_middl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
- link right_hand_ring_proximal: geometry collision mesh filename=../meshes/end_effector/inspire_hand/visual/index_ring_proxi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; visual mesh filename=../meshes/end_effector/inspire_hand/visual/index_ring_proxi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
- link right_hand_thumb_distal: geometry collision mesh filename=../meshes/end_effector/inspire_hand/visual/thumb_distal.glb; visual mesh filename=../meshes/end_effector/inspire_hand/visual/thumb_distal.glb
- link right_hand_thumb_metacarpal: geometry collision mesh filename=../meshes/end_effector/inspire_hand/visual/thumb_metacarpal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; visual mesh filename=../meshes/end_effector/inspire_hand/visual/thumb_metacarpal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
- link right_hand_thumb_metacarpal_base: geometry collision mesh filename=../meshes/end_effector/inspire_hand/visual/R_thumb_metacarp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; visual mesh filename=../meshes/end_effector/inspire_hand/visual/R_thumb_metacarp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
- link right_hand_thumb_proximal: geometry collision mesh filename=../meshes/end_effector/inspire_hand/visual/thumb_proximal.g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; visual mesh filename=../meshes/end_effector/inspire_hand/visual/thumb_proximal.g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
- link right_hand_wrist_base_link: geometry collision mesh filename=../meshes/end_effector/inspire_hand/visual/wrist_base_link.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; visual mesh filename=../meshes/end_effector/inspire_hand/visual/wrist_base_link.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
- link right_hand_wrist_link: geometry collision mesh filename=../meshes/end_effector/inspire_hand/visual/R_wrist_link.glb; visual mesh filename=../meshes/end_effector/inspire_hand/visual/R_wrist_link.glb
Joints:
- joint right_hand_thumb_IP_joint: mimic joint=right_hand_thumb_MCP_joint multiplier=0.888 offset=0 -> joint=right_hand_thumb_MCP_joint multiplier=0.5 offset=0
