Commit message: fixes

File: mani_skill/assets/robots/inspire_hand/RH56DFX-2LR/urdf/inspire_hand_left.urdf (robot description, URDF)
Before this commit: robot inspire_hand, 20 links, 19 joints
Links:
- link left_hand_hand_base_link: geometry collision mesh filename=../meshes/visual/L_hand_base_link.glb; visual mesh filename=../meshes/visual/L_hand_base_link.glb
- link left_hand_index_middle: geometry collision mesh filename=../meshes/visual/index_ring_middle.glb; visual mesh filename=../meshes/visual/index_ring_middle.glb
- link left_hand_index_proximal: geometry collision mesh filename=../meshes/visual/index_ring_proximal.glb; visual mesh filename=../meshes/visual/index_ring_proximal.glb
- link left_hand_middle_middle: geometry collision mesh filename=../meshes/visual/middle_middle.glb; visual mesh filename=../meshes/visual/middle_middle.glb
- link left_hand_middle_proximal: geometry collision mesh filename=../meshes/visual/middle_pinky_proximal.glb; visual mesh filename=../meshes/visual/middle_pinky_proximal.glb
- link left_hand_pinky_middle: geometry collision mesh filename=../meshes/visual/pinky_middle.glb; visual mesh filename=../meshes/visual/pinky_middle.glb
- link left_hand_pinky_proximal: geometry collision mesh filename=../meshes/visual/middle_pinky_proximal.glb; visual mesh filename=../meshes/visual/middle_pinky_proximal.glb
- link left_hand_ring_middle: geometry collision mesh filename=../meshes/visual/index_ring_middle.glb; visual mesh filename=../meshes/visual/index_ring_middle.glb
- link left_hand_ring_proximal: geometry collision mesh filename=../meshes/visual/index_ring_proximal.glb; visual mesh filename=../meshes/visual/index_ring_proximal.glb
- link left_hand_thumb_distal: geometry collision mesh filename=../meshes/visual/thumb_distal.glb; visual mesh filename=../meshes/visual/thumb_distal.glb
- link left_hand_thumb_metacarpal: geometry collision mesh filename=../meshes/visual/thumb_metacarpal.glb; visual mesh filename=../meshes/visual/thumb_metacarpal.glb
- link left_hand_thumb_metacarpal_base: geometry collision mesh filename=../meshes/visual/L_thumb_metacarpal_base.glb; visual mesh filename=../meshes/visual/L_thumb_metacarpal_base.glb
- link left_hand_thumb_proximal: geometry collision mesh filename=../meshes/visual/thumb_proximal.glb; visual mesh filename=../meshes/visual/thumb_proximal.glb
- link left_hand_wrist_base_link: geometry collision mesh filename=../meshes/visual/wrist_base_link.glb; visual mesh filename=../meshes/visual/wrist_base_link.glb
- link left_hand_wrist_link: geometry collision mesh filename=../meshes/visual/L_wrist_link.glb; visual mesh filename=../meshes/visual/L_wrist_link.glb
Joints:
- joint left_hand_index_PIP_joint: limit lower=-1.56 upper=0.04545 effort=1 velocity=0.5 -> lower=-1.5930946000000001 upper=0.04545 effort=1 velocity=0.5; mimic (none) -> joint=left_hand_index_MCP_joint multiplier=1.06399 offset=-0.16734800000000002
- joint left_hand_middle_PIP_joint: limit lower=-1.56 upper=0.04545 effort=1 velocity=0.5 -> lower=-1.5930946000000001 upper=0.04545 effort=1 velocity=0.5; mimic (none) -> joint=left_hand_middle_MCP_joint multiplier=1.06399 offset=-0.16734800000000002
- joint left_hand_pinky_PIP_joint: limit lower=-1.56 upper=0.04545 effort=1 velocity=0.5 -> lower=-1.5930946000000001 upper=0.04545 effort=1 velocity=0.5; mimic (none) -> joint=left_hand_pinky_MCP_joint multiplier=1.06399 offset=-0.16734800000000002
- joint left_hand_ring_PIP_joint: limit lower=-1.56 upper=0.04545 effort=1 velocity=0.5 -> lower=-1.5930946000000001 upper=0.04545 effort=1 velocity=0.5; mimic (none) -> joint=left_hand_ring_MCP_joint multiplier=1.06399 offset=-0.16734800000000002
- joint left_hand_thumb_IP_joint: mimic (none) -> joint=left_hand_thumb_MCP_joint multiplier=0.5 offset=0
- joint left_hand_thumb_MCP_joint: mimic (none) -> joint=left_hand_thumb_CMC_pitch_joint multiplier=1.3333333333333335 offset=-0.08144869842640205

File: mani_skill/assets/robots/inspire_hand/RH56DFX-2LR/urdf/inspire_hand_right.urdf (robot description, URDF)
Before this commit: robot inspire_hand, 20 links, 19 joints
Links:
- link right_hand_hand_base_link: geometry collision mesh filename=../meshes/visual/R_hand_base_link.glb; visual mesh filename=../meshes/visual/R_hand_base_link.glb
- link right_hand_index_middle: geometry collision mesh filename=../meshes/visual/index_ring_middle.glb; visual mesh filename=../meshes/visual/index_ring_middle.glb
- link right_hand_index_proximal: geometry collision mesh filename=../meshes/visual/index_ring_proximal.glb; visual mesh filename=../meshes/visual/index_ring_proximal.glb
- link right_hand_middle_middle: geometry collision mesh filename=../meshes/visual/middle_middle.glb; visual mesh filename=../meshes/visual/middle_middle.glb
- link right_hand_middle_proximal: geometry collision mesh filename=../meshes/visual/middle_pinky_proximal.glb; visual mesh filename=../meshes/visual/middle_pinky_proximal.glb
- link right_hand_pinky_middle: geometry collision mesh filename=../meshes/visual/pinky_middle.glb; visual mesh filename=../meshes/visual/pinky_middle.glb
- link right_hand_pinky_proximal: geometry collision mesh filename=../meshes/visual/middle_pinky_proximal.glb; visual mesh filename=../meshes/visual/middle_pinky_proximal.glb
- link right_hand_ring_middle: geometry collision mesh filename=../meshes/visual/index_ring_middle.glb; visual mesh filename=../meshes/visual/index_ring_middle.glb
- link right_hand_ring_proximal: geometry collision mesh filename=../meshes/visual/index_ring_proximal.glb; visual mesh filename=../meshes/visual/index_ring_proximal.glb
- link right_hand_thumb_distal: geometry collision mesh filename=../meshes/visual/thumb_distal.glb; visual mesh filename=../meshes/visual/thumb_distal.glb
- link right_hand_thumb_metacarpal: geometry collision mesh filename=../meshes/visual/thumb_metacarpal.glb; visual mesh filename=../meshes/visual/thumb_metacarpal.glb
- link right_hand_thumb_metacarpal_base: geometry collision mesh filename=../meshes/visual/R_thumb_metacarpal_base.glb; visual mesh filename=../meshes/visual/R_thumb_metacarpal_base.glb
- link right_hand_thumb_proximal: geometry collision mesh filename=../meshes/visual/thumb_proximal.glb; visual mesh filename=../meshes/visual/thumb_proximal.glb
- link right_hand_wrist_base_link: geometry collision mesh filename=../meshes/visual/wrist_base_link.glb; visual mesh filename=../meshes/visual/wrist_base_link.glb
- link right_hand_wrist_link: geometry collision mesh filename=../meshes/visual/R_wrist_link.glb; visual mesh filename=../meshes/visual/R_wrist_link.glb

File: mani_skill/assets/robots/inspire_hand/RH56DFX-2LR/urdf/inspire_hand_right_floating.urdf (robot description, URDF)
Before this commit: robot inspire_hand, 26 links, 25 joints
Links:
- link right_hand_hand_base_link: geometry collision mesh filename=../meshes/visual/R_hand_base_link.glb; visual mesh filename=../meshes/visual/R_hand_base_link.glb
- link right_hand_index_middle: geometry collision mesh filename=../meshes/visual/index_ring_middle.glb; visual mesh filename=../meshes/visual/index_ring_middle.glb
- link right_hand_index_proximal: geometry collision mesh filename=../meshes/visual/index_ring_proximal.glb; visual mesh filename=../meshes/visual/index_ring_proximal.glb
- link right_hand_middle_middle: geometry collision mesh filename=../meshes/visual/middle_middle.glb; visual mesh filename=../meshes/visual/middle_middle.glb
- link right_hand_middle_proximal: geometry collision mesh filename=../meshes/visual/middle_pinky_proximal.glb; visual mesh filename=../meshes/visual/middle_pinky_proximal.glb
- link right_hand_pinky_middle: geometry collision mesh filename=../meshes/visual/pinky_middle.glb; visual mesh filename=../meshes/visual/pinky_middle.glb
- link right_hand_pinky_proximal: geometry collision mesh filename=../meshes/visual/middle_pinky_proximal.glb; visual mesh filename=../meshes/visual/middle_pinky_proximal.glb
- link right_hand_ring_middle: geometry collision mesh filename=../meshes/visual/index_ring_middle.glb; visual mesh filename=../meshes/visual/index_ring_middle.glb
- link right_hand_ring_proximal: geometry collision mesh filename=../meshes/visual/index_ring_proximal.glb; visual mesh filename=../meshes/visual/index_ring_proximal.glb
- link right_hand_thumb_distal: geometry collision mesh filename=../meshes/visual/thumb_distal.glb; visual mesh filename=../meshes/visual/thumb_distal.glb
- link right_hand_thumb_metacarpal: geometry collision mesh filename=../meshes/visual/thumb_metacarpal.glb; visual mesh filename=../meshes/visual/thumb_metacarpal.glb
- link right_hand_thumb_metacarpal_base: geometry collision mesh filename=../meshes/visual/R_thumb_metacarpal_base.glb; visual mesh filename=../meshes/visual/R_thumb_metacarpal_base.glb
- link right_hand_thumb_proximal: geometry collision mesh filename=../meshes/visual/thumb_proximal.glb; visual mesh filename=../meshes/visual/thumb_proximal.glb
- link right_hand_wrist_base_link: geometry collision mesh filename=../meshes/visual/wrist_base_link.glb; visual mesh filename=../meshes/visual/wrist_base_link.glb
- link right_hand_wrist_link: geometry collision mesh filename=../meshes/visual/R_wrist_link.glb; visual mesh filename=../meshes/visual/R_wrist_link.glb
