Commit message: work

File: mani_skill/assets/robots/inspire_hand/RH56DFX-2LR/urdf/inspire_hand_right.urdf (robot description, URDF)
Before this commit: robot inspire_hand, 20 links, 19 joints
Links:
- link right_hand_hand_base_link: geometry collision mesh filename=../meshes/end_effector/inspire_hand/visual/R_hand_base_link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; visual mesh filename=../meshes/end_effector/inspire_hand/visual/R_hand_base_link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
- link right_hand_index_middle: geometry collision mesh filename=../meshes/end_effector/inspire_hand/visual/index_ring_middl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; visual mesh filename=../meshes/end_effector/inspire_hand/visual/index_ring_middl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
- link right_hand_index_proximal: geometry collision mesh filename=../meshes/end_effector/inspire_hand/visual/index_ring_proxi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; visual mesh filename=../meshes/end_effector/inspire_hand/visual/index_ring_proxi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
- link right_hand_middle_middle: geometry collision mesh filename=../meshes/end_effector/inspire_hand/visual/middle_middle.glb; visual mesh filename=../meshes/end_effector/inspire_hand/visual/middle_middle.glb
- link right_hand_middle_proximal: geometry collision mesh filename=../meshes/end_effector/inspire_hand/visual/middle_pinky_pro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; visual mesh filename=../meshes/end_effector/inspire_hand/visual/middle_pinky_pro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
- link right_hand_pinky_middle: geometry collision mesh filename=../meshes/end_effector/inspire_hand/visual/pinky_middle.glb; visual mesh filename=../meshes/end_effector/inspire_hand/visual/pinky_middle.glb
- link right_hand_pinky_proximal: geometry collision mesh filename=../meshes/end_effector/inspire_hand/visual/middle_pinky_pro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; visual mesh filename=../meshes/end_effector/inspire_hand/visual/middle_pinky_pro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
- link right_hand_ring_middle: geometry collision mesh filename=../meshes/end_effector/inspire_hand/visual/index_ring_middl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; visual mesh filename=../meshes/end_effector/inspire_hand/visual/index_ring_middl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
- link right_hand_ring_proximal: geometry collision mesh filename=../meshes/end_effector/inspire_hand/visual/index_ring_proxi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; visual mesh filename=../meshes/end_effector/inspire_hand/visual/index_ring_proxi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
- link right_hand_thumb_distal: geometry collision mesh filename=../meshes/end_effector/inspire_hand/visual/thumb_distal.glb; visual mesh filename=../meshes/end_effector/inspire_hand/visual/thumb_distal.glb
- link right_hand_thumb_metacarpal: geometry collision mesh filename=../meshes/end_effector/inspire_hand/visual/thumb_metacarpal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; visual mesh filename=../meshes/end_effector/inspire_hand/visual/thumb_metacarpal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
- link right_hand_thumb_metacarpal_base: geometry collision mesh filename=../meshes/end_effector/inspire_hand/visual/R_thumb_metacarp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; visual mesh filename=../meshes/end_effector/inspire_hand/visual/R_thumb_metacarp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
- link right_hand_thumb_proximal: geometry collision mesh filename=../meshes/end_effector/inspire_hand/visual/thumb_proximal.g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; visual mesh filename=../meshes/end_effector/inspire_hand/visual/thumb_proximal.g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
- link right_hand_wrist_base_link: geometry collision mesh filename=../meshes/end_effector/inspire_hand/visual/wrist_base_link.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; visual mesh filename=../meshes/end_effector/inspire_hand/visual/wrist_base_link.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
- link right_hand_wrist_link: geometry collision mesh filename=../meshes/end_effector/inspire_hand/visual/R_wrist_link.glb; visual mesh filename=../meshes/end_effector/inspire_hand/visual/R_wrist_link.glb
Joints:
- joint right_hand_index_PIP_joint: limit lower=-1.56 upper=0.04545 effort=1 velocity=0.5 -> lower=-1.5930946000000001 upper=0.04545 effort=1 velocity=0.5; mimic (none) -> joint=right_hand_index_MCP_joint multiplier=1.06399 offset=-0.16734800000000002
- joint right_hand_middle_PIP_joint: limit lower=-1.56 upper=0.04545 effort=1 velocity=0.5 -> lower=-1.5930946000000001 upper=0.04545 effort=1 velocity=0.5; mimic (none) -> joint=right_hand_middle_MCP_joint multiplier=1.06399 offset=-0.16734800000000002
- joint right_hand_pinky_PIP_joint: limit lower=-1.56 upper=0.04545 effort=1 velocity=0.5 -> lower=-1.5930946000000001 upper=0.04545 effort=1 velocity=0.5; mimic (none) -> joint=right_hand_pinky_MCP_joint multiplier=1.06399 offset=-0.16734800000000002
- joint right_hand_ring_PIP_joint: limit lower=-1.56 upper=0.04545 effort=1 velocity=0.5 -> lower=-1.5930946000000001 upper=0.04545 effort=1 velocity=0.5; mimic (none) -> joint=right_hand_ring_MCP_joint multiplier=1.06399 offset=-0.16734800000000002
- joint right_hand_thumb_IP_joint: mimic (none) -> joint=right_hand_thumb_MCP_joint multiplier=0.5 offset=0
- joint right_hand_thumb_MCP_joint: mimic (none) -> joint=right_hand_thumb_CMC_pitch_joint multiplier=1.3333333333333335 offset=-0.08144869842640205

Commit message: [BugFix] Fix some NaN issues with physx backend for fixed tendon modelled robots. (#1080)
* work

* more stable

* work

* work

* work

* fixes

* files

* update robot docs

* refactor

* refactor

File: mani_skill/assets/robots/inspire_hand/RH56DFX-2LR/urdf/inspire_hand_right.urdf (robot description, URDF)
Before this commit: robot inspire_hand, 26 links, 25 joints
Links:
- removed link root
- removed link root_arm_1_link_1
- removed link root_arm_1_link_2
- removed link root_arm_1_link_3
- removed link root_arm_1_link_4
- removed link root_arm_1_link_5
- link right_hand_hand_base_link: geometry collision mesh filename=../meshes/visual/R_hand_base_link.glb; visual mesh filename=../meshes/visual/R_hand_base_link.glb
- link right_hand_index_middle: geometry collision mesh filename=../meshes/visual/index_ring_middle.glb; visual mesh filename=../meshes/visual/index_ring_middle.glb
- link right_hand_index_proximal: geometry collision mesh filename=../meshes/visual/index_ring_proximal.glb; visual mesh filename=../meshes/visual/index_ring_proximal.glb
- link right_hand_middle_middle: geometry collision mesh filename=../meshes/visual/middle_middle.glb; visual mesh filename=../meshes/visual/middle_middle.glb
- link right_hand_middle_proximal: geometry collision mesh filename=../meshes/visual/middle_pinky_proximal.glb; visual mesh filename=../meshes/visual/middle_pinky_proximal.glb
- link right_hand_pinky_middle: geometry collision mesh filename=../meshes/visual/pinky_middle.glb; visual mesh filename=../meshes/visual/pinky_middle.glb
- link right_hand_pinky_proximal: geometry collision mesh filename=../meshes/visual/middle_pinky_proximal.glb; visual mesh filename=../meshes/visual/middle_pinky_proximal.glb
- link right_hand_ring_middle: geometry collision mesh filename=../meshes/visual/index_ring_middle.glb; visual mesh filename=../meshes/visual/index_ring_middle.glb
- link right_hand_ring_proximal: geometry collision mesh filename=../meshes/visual/index_ring_proximal.glb; visual mesh filename=../meshes/visual/index_ring_proximal.glb
- link right_hand_thumb_distal: geometry collision mesh filename=../meshes/visual/thumb_distal.glb; visual mesh filename=../meshes/visual/thumb_distal.glb
- link right_hand_thumb_metacarpal: geometry collision mesh filename=../meshes/visual/thumb_metacarpal.glb; visual mesh filename=../meshes/visual/thumb_metacarpal.glb
- link right_hand_thumb_metacarpal_base: geometry collision mesh filename=../meshes/visual/R_thumb_metacarpal_base.glb; visual mesh filename=../meshes/visual/R_thumb_metacarpal_base.glb
- link right_hand_thumb_proximal: geometry collision mesh filename=../meshes/visual/thumb_proximal.glb; visual mesh filename=../meshes/visual/thumb_proximal.glb
- link right_hand_wrist_base_link: geometry collision mesh filename=../meshes/visual/wrist_base_link.glb; visual mesh filename=../meshes/visual/wrist_base_link.glb
- link right_hand_wrist_link: geometry collision mesh filename=../meshes/visual/R_wrist_link.glb; visual mesh filename=../meshes/visual/R_wrist_link.glb
Joints:
- removed joint root_x_axis_joint
- removed joint root_x_rot_joint
- removed joint root_y_axis_joint
- removed joint root_y_rot_joint
- removed joint root_z_axis_joint
- removed joint root_z_rot_joint
- joint right_hand_index_PIP_joint: limit lower=-1.56 upper=0.04545 effort=1 velocity=0.5 -> lower=-1.5930946000000001 upper=0.04545 effort=1 velocity=0.5; mimic (none) -> joint=right_hand_index_MCP_joint multiplier=1.06399 offset=-0.16734800000000002
- joint right_hand_middle_PIP_joint: limit lower=-1.56 upper=0.04545 effort=1 velocity=0.5 -> lower=-1.5930946000000001 upper=0.04545 effort=1 velocity=0.5; mimic (none) -> joint=right_hand_middle_MCP_joint multiplier=1.06399 offset=-0.16734800000000002
- joint right_hand_pinky_PIP_joint: limit lower=-1.56 upper=0.04545 effort=1 velocity=0.5 -> lower=-1.5930946000000001 upper=0.04545 effort=1 velocity=0.5; mimic (none) -> joint=right_hand_pinky_MCP_joint multiplier=1.06399 offset=-0.16734800000000002
- joint right_hand_ring_PIP_joint: limit lower=-1.56 upper=0.04545 effort=1 velocity=0.5 -> lower=-1.5930946000000001 upper=0.04545 effort=1 velocity=0.5; mimic (none) -> joint=right_hand_ring_MCP_joint multiplier=1.06399 offset=-0.16734800000000002
- joint right_hand_thumb_IP_joint: mimic (none) -> joint=right_hand_thumb_MCP_joint multiplier=0.5 offset=0
- joint right_hand_thumb_MCP_joint: mimic (none) -> joint=right_hand_thumb_CMC_pitch_joint multiplier=1.3333333333333335 offset=-0.08144869842640205

File: mani_skill/assets/robots/inspire_hand/RH56DFX-2LR/urdf/inspire_hand_right_floating.urdf (robot description, URDF)
Before this commit: robot inspire_hand, 20 links, 19 joints
Links:
- added link root, mass 0
- added link root_arm_1_link_1, mass 0
- added link root_arm_1_link_2, mass 0
- added link root_arm_1_link_3, mass 0
- added link root_arm_1_link_4, mass 0
- added link root_arm_1_link_5, mass 0
- link right_hand_hand_base_link: geometry collision mesh filename=../meshes/visual/R_hand_base_link.glb; visual mesh filename=../meshes/visual/R_hand_base_link.glb
- link right_hand_index_middle: geometry collision mesh filename=../meshes/visual/index_ring_middle.glb; visual mesh filename=../meshes/visual/index_ring_middle.glb
- link right_hand_index_proximal: geometry collision mesh filename=../meshes/visual/index_ring_proximal.glb; visual mesh filename=../meshes/visual/index_ring_proximal.glb
- link right_hand_middle_middle: geometry collision mesh filename=../meshes/visual/middle_middle.glb; visual mesh filename=../meshes/visual/middle_middle.glb
- link right_hand_middle_proximal: geometry collision mesh filename=../meshes/visual/middle_pinky_proximal.glb; visual mesh filename=../meshes/visual/middle_pinky_proximal.glb
- link right_hand_pinky_middle: geometry collision mesh filename=../meshes/visual/pinky_middle.glb; visual mesh filename=../meshes/visual/pinky_middle.glb
- link right_hand_pinky_proximal: geometry collision mesh filename=../meshes/visual/middle_pinky_proximal.glb; visual mesh filename=../meshes/visual/middle_pinky_proximal.glb
- link right_hand_ring_middle: geometry collision mesh filename=../meshes/visual/index_ring_middle.glb; visual mesh filename=../meshes/visual/index_ring_middle.glb
- link right_hand_ring_proximal: geometry collision mesh filename=../meshes/visual/index_ring_proximal.glb; visual mesh filename=../meshes/visual/index_ring_proximal.glb
- link right_hand_thumb_distal: geometry collision mesh filename=../meshes/visual/thumb_distal.glb; visual mesh filename=../meshes/visual/thumb_distal.glb
- link right_hand_thumb_metacarpal: geometry collision mesh filename=../meshes/visual/thumb_metacarpal.glb; visual mesh filename=../meshes/visual/thumb_metacarpal.glb
- link right_hand_thumb_metacarpal_base: geometry collision mesh filename=../meshes/visual/R_thumb_metacarpal_base.glb; visual mesh filename=../meshes/visual/R_thumb_metacarpal_base.glb
- link right_hand_thumb_proximal: geometry collision mesh filename=../meshes/visual/thumb_proximal.glb; visual mesh filename=../meshes/visual/thumb_proximal.glb
- link right_hand_wrist_base_link: geometry collision mesh filename=../meshes/visual/wrist_base_link.glb; visual mesh filename=../meshes/visual/wrist_base_link.glb
- link right_hand_wrist_link: geometry collision mesh filename=../meshes/visual/R_wrist_link.glb; visual mesh filename=../meshes/visual/R_wrist_link.glb
Joints:
- added joint root_x_axis_joint: type prismatic, parent root, child root_arm_1_link_1, axis 1 0 0, limit lower=-20 upper=20 effort=100 velocity=0.50
- added joint root_x_rot_joint: type revolute, parent root_arm_1_link_3, child root_arm_1_link_4, axis 1 0 0, limit lower=-20 upper=20 effort=100 velocity=0.50
- added joint root_y_axis_joint: type prismatic, parent root_arm_1_link_1, child root_arm_1_link_2, axis 0 1 0, limit lower=-20 upper=20 effort=100 velocity=0.50
- added joint root_y_rot_joint: type revolute, parent root_arm_1_link_4, child root_arm_1_link_5, axis 0 1 0, limit lower=-20 upper=20 effort=100 velocity=0.50
- added joint root_z_axis_joint: type prismatic, parent root_arm_1_link_2, child root_arm_1_link_3, axis 0 0 1, limit lower=-20 upper=20 effort=100 velocity=0.50
- added joint root_z_rot_joint: type revolute, parent root_arm_1_link_5, child right_hand_wrist_base_link, axis 0 0 1, limit lower=-20 upper=20 effort=100 velocity=0.50
- joint right_hand_index_PIP_joint: limit lower=-1.56 upper=0.04545 effort=1 velocity=0.5 -> lower=-1.5930946000000001 upper=0.04545 effort=1 velocity=0.5; mimic (none) -> joint=right_hand_index_MCP_joint multiplier=1.06399 offset=-0.16734800000000002
- joint right_hand_middle_PIP_joint: limit lower=-1.56 upper=0.04545 effort=1 velocity=0.5 -> lower=-1.5930946000000001 upper=0.04545 effort=1 velocity=0.5; mimic (none) -> joint=right_hand_middle_MCP_joint multiplier=1.06399 offset=-0.16734800000000002
- joint right_hand_pinky_PIP_joint: limit lower=-1.56 upper=0.04545 effort=1 velocity=0.5 -> lower=-1.5930946000000001 upper=0.04545 effort=1 velocity=0.5; mimic (none) -> joint=right_hand_pinky_MCP_joint multiplier=1.06399 offset=-0.16734800000000002
- joint right_hand_ring_PIP_joint: limit lower=-1.56 upper=0.04545 effort=1 velocity=0.5 -> lower=-1.5930946000000001 upper=0.04545 effort=1 velocity=0.5; mimic (none) -> joint=right_hand_ring_MCP_joint multiplier=1.06399 offset=-0.16734800000000002
- joint right_hand_thumb_IP_joint: mimic (none) -> joint=right_hand_thumb_MCP_joint multiplier=0.5 offset=0
- joint right_hand_thumb_MCP_joint: mimic (none) -> joint=right_hand_thumb_CMC_pitch_joint multiplier=1.3333333333333335 offset=-0.08144869842640205
