Commit message: fixed convex mesh grasp bug

File: mani_skill/assets/robots/so101/so101.urdf (robot description, URDF)
Before this commit: robot so101_new_calib, 8 links, 7 joints
Links:
- link base_link: geometry collision mesh filename=meshes/base_motor_holder_so101_v1_convex.obj; collision mesh filename=meshes/base_so101_v2_convex.obj
- link gripper_link: geometry collision mesh filename=meshes/Fixed_part_1.obj; collision mesh filename=meshes/Fixed_part_2.obj
- link lower_arm_link: geometry collision mesh filename=meshes/motor_holder_so101_wrist_v1_convex.obj; collision mesh filename=meshes/sts3215_03a_v1_convex.obj
- link moving_jaw_so101_v1_link: geometry collision mesh filename=meshes/moving_jaw_so101_v1_convex.obj; visual mesh filename=meshes/moving_jaw_so101_v1.stl
- link shoulder_link: geometry collision mesh filename=meshes/motor_holder_so101_base_v1_convex.obj; collision mesh filename=meshes/rotation_pitch_so101_v1_convex.obj
- link upper_arm_link: geometry collision mesh filename=meshes/sts3215_03a_v1_convex.obj; collision mesh filename=meshes/upper_arm_so101_v1_convex.obj
- link wrist_link: geometry collision mesh filename=meshes/sts3215_03a_no_horn_v1_convex.obj; collision mesh filename=meshes/wrist_roll_pitch_so101_v2_convex.obj
Joints:
- joint gripper: origin xyz=0.0202 0.0188 -0.0234 rpy=1.5708 -5.24284e-08 -1.41553e-15 -> xyz=0.0202 0.0188 -0.0234 rpy=1.5708 -1.5708 -1.41553e-15

Commit message: fixed contact issues, working ppo training

File: mani_skill/assets/robots/so101/so101.urdf (robot description, URDF)
Before this commit: robot so101_new_calib, 8 links, 7 joints
Links:
- added link finger1_tip
- added link finger2_tip
Joints:
- added joint finger1_tip_joint: type fixed, parent gripper_link, child finger1_tip, origin xyz=-0.01 -0.0 -0.086 rpy=0 0 0
- added joint finger2_tip_joint: type fixed, parent moving_jaw_so101_v1_link, child finger2_tip, origin xyz=-0.01 -0.064 0.02 rpy=0 0 0
- joint elbow_flex: limit lower=-1.69 upper=1.69 effort=10 velocity=10 -> lower=-1.69 upper=1.69 effort=0 velocity=10
- joint gripper: limit lower=-0.174533 upper=1.74533 effort=10 velocity=10 -> lower=-1.74533 upper=0.174533 effort=0 velocity=10
- joint shoulder_lift: limit lower=-1.74533 upper=1.74533 effort=10 velocity=10 -> lower=-1.74533 upper=1.74533 effort=0 velocity=10
- joint shoulder_pan: limit lower=-1.91986 upper=1.91986 effort=10 velocity=10 -> lower=-1.91986 upper=1.91986 effort=0 velocity=10
- joint wrist_flex: limit lower=-1.65806 upper=1.65806 effort=10 velocity=10 -> lower=-1.65806 upper=1.65806 effort=0 velocity=10
- joint wrist_roll: limit lower=-2.74385 upper=2.84121 effort=10 velocity=10 -> lower=-2.74385 upper=2.84121 effort=0 velocity=10

Commit message: SysID with real robot for SO101 tested

File: mani_skill/assets/robots/so101/so101.urdf (robot description, URDF)
Before this commit: robot so101_new_calib, 10 links, 9 joints
Joints:
- joint elbow_flex: limit lower=-1.69 upper=1.69 effort=0 velocity=10 -> lower=-1.70012 upper=1.7046 effort=0 velocity=10; origin xyz=-0.11257 -0.028 1.73763e-16 rpy=-3.63608e-16 8.74301e-16 1.5708 -> xyz=-0.11257 -0.028 1.73763e-16 rpy=-3.63608e-16 0.03 1.5708
- joint gripper: limit lower=-1.74533 upper=0.174533 effort=0 velocity=10 -> lower=-1.13778 upper=1.16081 effort=0 velocity=10; origin xyz=0.0202 0.0188 -0.0234 rpy=1.5708 -1.5708 -1.41553e-15 -> xyz=0.0202 0.0188 -0.0234 rpy=1.5708 -0.909 -1.41553e-15
- joint shoulder_lift: limit lower=-1.74533 upper=1.74533 effort=0 velocity=10 -> lower=-1.82736 upper=1.83346 effort=0 velocity=10; origin xyz=-0.0303992 -0.0182778 -0.0542 rpy=-1.5708 -1.5708 0 -> xyz=-0.0303992 -0.0182778 -0.0542 rpy=-1.5708 -1.728 0
- joint shoulder_pan: limit lower=-1.91986 upper=1.91986 effort=0 velocity=10 -> lower=-2.15967042 upper=2.03383 effort=0 velocity=10
- joint wrist_flex: limit lower=-1.65806 upper=1.65806 effort=0 velocity=10 -> lower=-1.81130 upper=1.80816 effort=0 velocity=10
- joint wrist_roll: limit lower=-2.74385 upper=2.84121 effort=0 velocity=10 -> lower=-2.93145 upper=2.92988 effort=0 velocity=10

Commit message: added fixed urdf with real agent

File: mani_skill/assets/robots/so101/so101.urdf (robot description, URDF)
Before this commit: robot so101_new_calib, 10 links, 9 joints
Joints:
- joint elbow_flex: origin xyz=-0.11257 -0.028 1.73763e-16 rpy=-3.63608e-16 0.03 1.5708 -> xyz=-0.11257 -0.028 1.73763e-16 rpy=-3.63608e-16 8.74301e-16 1.4408
- joint finger1_tip_joint: origin xyz=-0.01 -0.0 -0.086 rpy=0 0 0 -> xyz=-0.002 -0.0 -0.092 rpy=0 0 0
- joint finger2_tip_joint: origin xyz=-0.01 -0.064 0.02 rpy=0 0 0 -> xyz=-0.01 -0.077 0.02 rpy=0 0 0
- joint gripper: limit lower=-1.13778 upper=1.16081 effort=0 velocity=10 -> lower=-0.174533 upper=2.0944 effort=10 velocity=10; origin xyz=0.0202 0.0188 -0.0234 rpy=1.5708 -0.909 -1.41553e-15 -> xyz=0.0202 0.0188 -0.0234 rpy=1.5708 -5.24284e-08 -1.41553e-15
- joint shoulder_lift: origin xyz=-0.0303992 -0.0182778 -0.0542 rpy=-1.5708 -1.728 0 -> xyz=-0.0303992 -0.0182778 -0.0542 rpy=-1.5708 -1.6208 0.03
- joint shoulder_pan: origin xyz=0.0388353 -8.97657e-09 0.0624 rpy=3.14159 4.18253e-17 -3.14159 -> xyz=0.0388353 -8.97657e-09 0.0624 rpy=3.14159 4.18253e-17 -3.20159
- joint wrist_flex: origin xyz=-0.1349 0.0052 3.62355e-17 rpy=4.02456e-15 8.67362e-16 -1.5708 -> xyz=-0.1349 0.0052 3.62355e-17 rpy=4.02456e-15 8.67362e-16 -1.6708
- joint wrist_roll: origin xyz=5.55112e-17 -0.0611 0.0181 rpy=1.5708 0.0486795 3.14159 -> xyz=5.55112e-17 -0.0611 0.0181 rpy=1.5708 0 3.09159

Commit message: fix: urdf values, gripper mesh and rest qpos

File: mani_skill/assets/robots/so101/so101.urdf (robot description, URDF)
Before this commit: robot so101_new_calib, 10 links, 9 joints
Joints:
- joint elbow_flex: origin xyz=-0.11257 -0.028 1.73763e-16 rpy=-3.63608e-16 8.74301e-16 1.4408 -> xyz=-0.11257 -0.028 0 rpy=0 0 1.4408
- joint gripper: origin xyz=0.0202 0.0188 -0.0234 rpy=1.5708 -5.24284e-08 -1.41553e-15 -> xyz=0.0202 0.0188 -0.0234 rpy=1.5708 0 0
- joint shoulder_pan: origin xyz=0.0388353 -8.97657e-09 0.0624 rpy=3.14159 4.18253e-17 -3.20159 -> xyz=0.0388353 0 0.0624 rpy=3.14159 0 -3.20159
- joint wrist_flex: origin xyz=-0.1349 0.0052 3.62355e-17 rpy=4.02456e-15 8.67362e-16 -1.6708 -> xyz=-0.1349 0.0052 0 rpy=0 0 -1.6708
- joint wrist_roll: limit lower=-2.93145 upper=2.92988 effort=0 velocity=10 -> lower=-2.93145 upper=2.92988 effort=10 velocity=10; origin xyz=5.55112e-17 -0.0611 0.0181 rpy=1.5708 0 3.09159 -> xyz=0 -0.0611 0.0181 rpy=1.5708 0 3.09159
