Commit message: update assets

File: mani_skill/assets/robots/ability_hand/ability_hand_right_floating.urdf (robot description, URDF)
Before this commit: robot ability_hand, 24 links, 23 joints
Links:
- link index_L2: geometry collision mesh filename=meshes/collision/idx-F2_C.obj; collision sphere radius=0.007
