Commit message: [Feature] Add wrist camera mount and so100_wristcam robot variant for SO100
Add a fixed camera mount (camera_mount_link + camera_link, following the
existing panda_v3.urdf pattern) to the SO100 wrist and a new registered
so100_wristcam agent that provides a centered, downward-facing wrist camera
default that is usable for RL, as discussed in #1338. The mount links are
massless with no collision geometry so the arm's dynamics are unchanged, and
PickCube-v1 supports the new robot uid out of the box.

Closes #1338.

File: mani_skill/assets/robots/so100/so100.urdf (robot description, URDF)
Before this commit: robot SO_5DOF_ARM100_8j_URDF.SLDASM, 9 links, 8 joints
Links:
- added link camera_link
- added link camera_mount_link
Joints:
- added joint camera_link_joint: type fixed, parent camera_mount_link, child camera_link, origin xyz=0 0 0.015 rpy=0 1.309 1.5708
- added joint camera_mount_joint: type fixed, parent Wrist_Pitch_Roll, child camera_mount_link, origin xyz=0.02 -0.02 0.035 rpy=-1.5708 0 0
